File: Plaque_Leds_1.sch (KiCad schematic (older format))
At the start: 85 parts, among them J1 Conn_01x04

Commit message: jst coudé
Parts:
- J1: footprint Connector_JST:JST_XH_B4B-XH-A_1x04_P2.50mm_Vertical -> Connector_JST:JST_XH_S4B-XH-A_1x04_P2.50mm_Horizontal
Changed lines of the file:
@@
 F 0 "J1" H 5930 7392 50  0000 L CNN
 F 1 "Conn_01x04" H 5930 7301 50  0000 L CNN
-F 2 "Connector_JST:JST_XH_B4B-XH-A_1x04_P2.50mm_Vertical" H 5850 7400 50  0001 C CNN
+F 2 "Connector_JST:JST_XH_S4B-XH-A_1x04_P2.50mm_Horizontal" H 5850 7400 50  0001 C CNN
 F 3 "~" H 5850 7400 50  0001 C CNN
 	1    5850 7400
